File: traffic-light/traffic-light.sch (KiCad schematic (older format))
At the start: 11 parts, among them J1 Conn_01x04_Male

Commit message: traffic-light: add round edges, correct pin header, add silk screen
Parts:
- removed J1: Conn_01x04_Male, Connector_PinSocket_2.54mm:PinSocket_1x04_P2.54mm_Horizontal, symbol Connector:Conn_01x04_Male
- added J1: Conn_01x04_Female, Connector_PinHeader_2.54mm:PinHeader_1x04_P2.54mm_Horizontal, symbol Connector:Conn_01x04_Female
Connections:
- net at D1.1 (K), D2.1 (K), D3.1 (K): now also J1.1 (Pin_1)
- net at R1.2: now also J1.2 (Pin_2)
- net at R2.2: now also J1.3 (Pin_3)
- net at R3.2: now also J1.4 (Pin_4)
Changed lines of the file:
@@
-$EndComp
-$Comp
-L Connector:Conn_01x04_Male J1
-U 1 1 616754D6
-P 2700 3350
-F 0 "J1" H 2808 3631 50  0000 C CNN
-F 1 "Conn_01x04_Male" H 2808 3540 50  0000 C CNN
-F 2 "Connector_PinSocket_2.54mm:PinSocket_1x04_P2.54mm_Horizontal" H 2700 3350 50  0001 C CNN
-F 3 "~" H 2700 3350 50  0001 C CNN
-	1    2700 3350
-	1    0    0    -1
 $EndComp
 $Comp
@@
 	4500 3700 4500 3350
 Connection ~ 4500 3350
+$Comp
+L Connector:Conn_01x04_Female J1
+U 1 1 616EB7B9
+P 3050 3300
+F 0 "J1" H 2950 3850 50  0000 L CNN
+F 1 "Conn_01x04_Female" H 2650 3750 50  0000 L CNN
+F 2 "Connector_PinHeader_2.54mm:PinHeader_1x04_P2.54mm_Horizontal" H 3050 3300 50  0001 C CNN
+F 3 "~" H 3050 3300 50  0001 C CNN
+	1    3050 3300
+	1    0    0    -1
+$EndComp
 Wire Wire Line
-	2900 3250 3150 3250
+	4500 3700 4500 3800
+Connection ~ 4500 3700
 Wire Wire Line
-	3150 3250 3150 2700
+	2600 3800 2600 3200
 Wire Wire Line
-	3150 2700 4500 2700
+	2600 3200 2850 3200
 Wire Wire Line
-	4500 2700 4500 3000
-Connection ~ 4500 3000
+	2600 3800 4500 3800
 Wire Wire Line
-	2900 3350 3200 3350
+	3500 3000 3500 3300
 Wire Wire Line
-	3200 3350 3200 3000
+	3500 3300 2850 3300
 Wire Wire Line
-	3200 3000 3500 3000
+	3500 3350 2850 3350
 Wire Wire Line
-	2900 3450 3250 3450
+	2850 3350 2850 3400
 Wire Wire Line
-	3250 3450 3250 3350
+	3500 3700 2850 3700
 Wire Wire Line
-	3250 3350 3500 3350
-Wire Wire Line
-	2900 3550 3300 3550
-Wire Wire Line
-	3300 3550 3300 3700
-Wire Wire Line
-	3300 3700 3500 3700
+	2850 3700 2850 3500
 $EndSCHEMATC
